File: Hardware/TMP117/Datalogger2039_TMP117_adapter/Datalogger2039_TMP117_adapter.kicad_pcb (KiCad board)
At the start: 2 copper layers, 89.9 x 49.8 mm, 134 parts, among them J1 To_MCU, Q1 AO3401A, Q2 AO3401A, Q3 AO3401A, Q4 AO3401A, Q5 AO3401A, Q6 AO3401A, Q7 AO3401A, Q8 AO3401A, U1 TCA9548APWR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

Commit message: Update
Parts:
- moved JP7 85.8 mm to (156.7, 115.2)
- moved R23 83.0 mm to (158.0, 110.9), turned to -90 degrees
- moved R27 82.7 mm to (176.2, 110.8), turned to -90 degrees
- moved JP9 82.6 mm to (175.0, 115.3)
- moved R22 81.4 mm to (155.4, 110.9), turned to -90 degrees
- moved R26 80.2 mm to (173.7, 110.9), turned to -90 degrees
- moved JP5 62.1 mm to (138.9, 115.3)
- moved R19 62.0 mm to (140.2, 110.9), turned to -90 degrees
- moved R18 59.5 mm to (137.7, 110.9), turned to -90 degrees
- moved R11 44.8 mm to (137.3, 97.3), turned to 90 degrees
- moved I2C1 43.0 mm to (133.9, 94.8)
- moved R10 41.5 mm to (132.7, 98.5), turned to 90 degrees
- moved JP3 35.7 mm to (121.2, 115.1)
- moved R15 31.0 mm to (122.4, 110.7), turned to -90 degrees
- moved R14 29.9 mm to (119.9, 110.7), turned to -90 degrees
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Routing:
- net GND: track 101.7 -> 126.9 mm, vias 72 -> 104
- net Power7: track 91.1 -> 70.7 mm, vias 1 -> 3
- net Net-(D3-K): track 28.9 -> 39.3 mm
- net Net-(D5-K): track 29.4 -> 39.8 mm
- net Net-(D7-K): track 29.4 -> 39.7 mm
- net Net-(D9-K): track 29.3 -> 39.5 mm
- net Net-(D8-K): track 31.5 -> 41.7 mm
- net Alert1: track 19.8 -> 28.3 mm
- net Power4: track 27.6 -> 34.5 mm
- net Alert7: track 63.0 -> 69.7 mm
- net Power6: track 59.9 -> 65.6 mm
- net Alert6: track 50.6 -> 56.1 mm
- net Alert3: track 28.9 -> 33.3 mm
- net Alert5: track 47.6 -> 51.8 mm
- net VCC: track 159.8 -> 163.9 mm, vias 7 -> 8
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