File: Hardware/TMP117/Datalogger2039_TMP117_adapter/Datalogger2039_TMP117_adapter.kicad_sch (KiCad schematic)
At the start: 22 parts, among them J1 To_MCU, U1 TCA9548APWR, U10 PCF8575MS/TR

Commit message: Update
Other:
- company: (none) -> RTEK1000
- title: (none) -> Datalogger 2039 TMP117 Adapter
Changed lines of the file:
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@@
 (kicad_sch (version 20230121) (generator eeschema)
   (paper "A4")
+  (title_block
+    (title "Datalogger 2039 TMP117 Adapter")
+    (date "2023-07-09")
+    (rev "1.0")
+    (company "RTEK1000")
+  )
   (junction (at 72.39 31.75) (diameter 0) (color 0 0 0 0)
   )
