File: Hardware/TMP117/TMP117_Custom_Board/TMP117_custom_board/TMP117_custom_board.kicad_sch (KiCad schematic)
At the start: 14 parts, among them J1 Conn_01x06

Commit message: Update
Other:
- company: (none) -> RTEK1000
- title: (none) -> TMP117 Custom Board
Changed lines of the file:
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@@
 (kicad_sch (version 20230121) (generator eeschema)
   (paper "A4")
+  (title_block
+    (title "TMP117 Custom Board")
+    (date "2023-07-09")
+    (rev "1.0")
+    (company "RTEK1000")
+  )
   (junction (at 164.465 140.97) (diameter 0) (color 0 0 0 0)
   )
